File: Board/Carnivore2.kicad_pcb (KiCad board)
At the start: 2 copper layers, 99 x 65.6 mm, 132 parts, among them J1 Conn_01x02_Pin, J2 Conn_01x03_Pin, U1 EP2C8Q208C8N, U2 MX29LV640ETTI-70G, U3 RMLV1616AGSA-5S#KA0, U4 M25P80-VMN3TPB, U5 PCM5101APWR, U6 AT93C46DN-SH-T, U7 SG3225CAN 50.0000M-TJGA6, U9 PCM1808PWR, X1 EDGE50/MSX, X2 302-S101, X3 302-S101

Commit message: Some last details
Parts:
- added C18: 100nF, Capacitor_SMD:C_0603_1608Metric, B.Cu at (141.7, 107.2)
- added C19: 100nF, Capacitor_SMD:C_0603_1608Metric, F.Cu at (166.7, 86.3)
- added C20: 100nF, Capacitor_SMD:C_0603_1608Metric, F.Cu at (152.1, 82.5)
- C1, C105, C2, C205, C22, C23, C26, C28, C29, C3, C4: value 10uF 16V -> 10uF 10V
- C103, C203: value 10uF 16V -> 1uF 10V
- R103, R203: value 4.7k -> 75E
- X2, X3: footprint Library:HDR2X5 -> Library:302-S101
- moved C6 8.39 mm to (155.0, 110.7), turned to 0 degrees
- moved R46 1.40 mm to (190.7, 74.4)
- moved R44 1.31 mm to (168.3, 86.3)
- moved X2 1.30 mm to (178.1, 76.1)
- moved C15 1.00 mm to (170.7, 85.3)
- moved C14 0.97 mm to (170.7, 87.1)
- moved R64 0.97 mm to (110.1, 93.9)
- moved C8 0.95 mm to (155.0, 112.3)
Connections:
- C26 pad 2: Net-(C26-PLUS) -> /VCC3.3A
- C27 pad 2: Net-(C26-PLUS) -> /VCC3.3A
- U5 pad 1: Net-(C26-PLUS) -> /VCC3.3A
Routing:
- net /VCC3.3A: track 27.5 -> 45.0 mm, vias 2 -> 3
- net /GND: track 1017.3 -> 1031.2 mm
- net Net-(C26-PLUS): track 13.4 -> 0.00 mm, vias 1 -> 0
- net /VCC1.2: track 161.5 -> 166.7 mm
- net Net-(U1C-CONF_DONE): track 60.0 -> 62.6 mm
- net Net-(U1D-VCCA_PLL2): track 6.58 -> 8.67 mm
- net /NCONFIG: track 77.4 -> 79.3 mm
- net /ASDO: track 71.8 -> 73.1 mm, vias 2 -> 3
- net /VCC3.3: track 472.6 -> 473.3 mm
- net Net-(C23-PLUS): track 19.7 -> 18.9 mm
- net /NCSO: track 71.4 -> 72.2 mm
- net /NCE: track 86.6 -> 86.1 mm, vias 2 -> 1
Other:
- board text added: "Carnivore v3.0 MSX Cartridge RBSC/SHS 2024"
- board text removed: "Carnivore v3.0 MSX Cartridge RBSC/TICM 2024"

Commit message: Last update before ordering PCB
Parts:
- moved C103 0.81 mm to (125.3, 81.9)
- moved C203 0.81 mm to (125.3, 79.4)
- moved X1 0.44 mm to (179.6, 130.6)
Routing:
- net Net-(C203-MINUS): track 17.2 -> 18.0 mm
- net Net-(C103-MINUS): track 7.76 -> 8.54 mm
- net Net-(C103-PLUS): track 3.80 -> 3.27 mm
