File: Board/Carnivore2.kicad_sch (KiCad schematic)
At the start: 147 parts, among them T1 NPN, T2 PNP, T3 NPN, T4 NPN, T5 NPN, T6 PNP, U1 EP2C5Q208C8, U2 M29W640GB_TSOP48, U3 CY62167DV30, U4 EPCS4SI8, U5 YAC516-E, U6 93C46DSM, U7 SG-310, X1 EDGE50/MSX, X2 HEADER_5X2, X3 HEADER_5X2

Commit message: Schematic and pcb conversion cleanup and rework
Parts:
- added H1, H2: MountingHole, symbol Mechanical:MountingHole
- added J1: Conn_01x02_Pin, JUMPER_1, symbol Connector:Conn_01x02_Pin
- added TP1, TP2: TestPoint, symbol Connector:TestPoint
- added U8: DNI, Oscillator:Oscillator_SMD_TXC_7C-4Pin_5.0x3.2mm_HandSoldering, symbol Sheet1-altium-import:root_0_SG-310
- AU1, AU2: value 4558D -> ~; footprint SOP8 -> 4558D_1
- AX1: value ST-222 -> {Value}; footprint ST-222 -> ST-222_1
- C1, C2, C22, C23, C26, C28, C3, C4: value CAP100RP -> 10mk; footprint CAP100RP -> C_1812_1
- C10, C11, C12, C13, C14, C15, C16, C17, C18, C19, C24, C25, C27, C30, C5, C6, C7, C8, C9: value C_0805 -> 0.1mk; footprint C0805_133B -> C_0603_1
- C101, C102, C201, C202: value C_0805 -> 1n; footprint C0805_133B -> C_0603_1
- C103, C105, C203, C205: value CAP100RP -> 4.7mk 25v; footprint CAP100RP -> C_1206_1
- C104, C204: value C_0805 -> 390p; footprint C0805_133B -> C_0603_1
- C20, C21: value CAP100RP -> 100mk 16v; footprint CAP100RP -> C_1812_1
- C29: value CAP100RP -> 22mk; footprint CAP100RP -> C_1812_1
- D1, D2: value DIODE -> D9; footprint (none) -> DIODE_1N4148_1
- D3, D4, D5, D6: value DIODE -> 1N4148; footprint (none) -> DIODE_1N4148_1
- LED1: value LED -> ~; footprint LED100 -> C_0603_1
- R10, R11, R12, R13, R14, R15, R16, R17, R18, R19, R2, R20, R21, R22, R23, R24, R25, R26, R27, R28, R29, R3, R30, R31, R32, R33, R34, R35, R36, R37, R38, R39, R4, R40, R41, R42, R5, R6, R7, R8, R9: value R_0805 -> 331; footprint R0805_102A -> C0603_1
- R101, R201, R46, R47, R48, R50, R52, R60, R65, R66: value R_0805 -> 10k; footprint R0805_102A -> R_0603_1
- R102, R103, R202, R203: value R_0805 -> 4.7k; footprint R0805_102A -> R_0603_1
- R104, R204: value R_0805 -> 100k; footprint R0805_102A -> R_0603_1
- R105, R205: value R_0805 -> 1.8k; footprint R0805_102A -> R_0603_1
- R106, R206, R51, R58, R59: value R_0805 -> 1k; footprint R0805_102A -> R_0603_1
- R43, R44, R54, R64: value R_0805 -> 10; footprint R0805_102A -> R_0603_1
- R45, R55, R56: value R_0805 -> 220; footprint R0805_102A -> R_0603_1
- R53, R61, R62, R63: value R_0805 -> 2.2k; footprint R0805_102A -> R_0603_1
- R57: value R_0805 -> 1K; footprint R0805_102A -> R_0603_1
- T1, T3, T4, T5: value NPN -> 2SC945; footprint (none) -> SOT-23(A1A2K)_1
- T2, T6: value PNP -> 2SA733; footprint (none) -> SOT-23(A1A2K)_1
- U1: value EP2C5Q208C8 -> ~; footprint PQFP208 -> EP2C5Q208C8_1
- U2: value M29W640GB_TSOP48 -> ~; footprint TSOP-48 -> M29W320DXXXNXX_1
- U3: value CY62167DV30 -> ~; footprint TSOP-48 -> CY62167DV30_1
- U4: value EPCS4SI8 -> ~; footprint SOIC8 -> EPCS4SI8_1
- U5: value YAC516-E -> ~; footprint SSOP24 -> YAC516-E_1
- U6: value 93C46DSM -> ~; footprint DIPSM8 -> M93C46MN1_1
- U7: value SG-310 -> 50 MHz; footprint SPXO_32_25 -> SG-310_1
- UCT1: value ADP3338 -> 1.2v; footprint SOT-223 -> ADP3338_1
- UCT2, UCT3: value ADP3338 -> 3.3v; footprint SOT-223 -> ADP3338_1
- X1: footprint EDGE50/100_350 -> EDGE50/MSX_1
- XC1: value CF-50-001 -> ~; footprint CP-50NN001 -> CF-50-001_1
Connections:
- net CONF_DONE: now also R47.2; no longer R47.1
- net GND: now also C1.1 (MINUS), C10.2, C102.2, C11.2, C12.1, C13.1, C14.2, C15.2, C17.2, C19.2, C2.1 (MINUS), C20.1 (MINUS), C201.1, C21.2 (PLUS), C22.1 (MINUS), C23.1 (MINUS), C26.1 (MINUS), C28.1 (MINUS), C29.1 (MINUS), C3.1 (MINUS), C4.1 (MINUS), C5.1, R50.1, T1.A2 (E), T3.K (C), T4.K (C), T5.K (C), J1.1 (Pin_1), U8.2 (GND); no longer C1.MINUS, C10.1, C102.1, C11.1, C12.2, C13.2, C14.1, C15.1, C17.1, C19.1, C2.MINUS, C20.MINUS, C201.2, C21.PLUS, C22.MINUS, C23.MINUS, C26.MINUS, C28.MINUS, C29.MINUS, C3.MINUS, C4.MINUS, C5.2, R50.2, T1.3 (E), T3.1 (C), T4.1 (C), T5.1 (C)
- net KN0: now also U8.3 (OUT)
- net NCONFIG: now also R48.2; no longer R48.1
- net RSW1: now also R15.1; no longer R17.1
- net RSW2: now also R25.1; no longer R6.1
- net RVPPE: now also R52.2; no longer R52.1
- net SLTSOUND: now also R106.2, R206.2, T4.A2 (E); no longer R106.1, R206.1, T4.3 (E)
- net SLT_A00: now also R9.1; no longer R29.1
- net SLT_A01: now also R36.1; no longer R28.1
- net SLT_A02: now also R8.1; no longer R31.1
- net SLT_A03: now also R37.1; no longer R30.1
- net SLT_A04: now also R7.1; no longer R33.1
- net SLT_A05: now also R38.1; no longer R32.1
- net SLT_A06: now also R12.1; no longer R23.1
- net SLT_A07: now also R33.1; no longer R22.1
- net SLT_A08: now also R11.1; no longer R25.1
- net SLT_A09: now also R31.1; no longer R18.1
- net SLT_A10: now also R13.1; no longer R21.1
- net SLT_A11: now also R32.1; no longer R20.1
- net SLT_A12: now also R34.1; no longer R24.1
- net SLT_A13: now also R10.1; no longer R27.1
- net SLT_A14: now also R35.1; no longer R26.1
- net SLT_A15: now also R14.1; no longer R19.1
- net SLT_CLC: now also R2.1; no longer R42.1
- net SLT_D0: now also R6.1; no longer R35.1
- net SLT_D1: now also R39.1; no longer R34.1
- net SLT_D2: now also R5.1; no longer R37.1
- net SLT_D3: now also R40.1; no longer R36.1
- net SLT_D4: now also R4.1; no longer R39.1
- net SLT_D5: now also R41.1; no longer R38.1
- net SLT_D6: now also R3.1; no longer R41.1
- net SLT_D7: now also R42.1; no longer R40.1
- net VCC: now also C4.2 (PLUS), C5.2; no longer C4.PLUS, C5.1
- net VCC+12: now also C19.1, T2.A2 (E); no longer C19.2, T2.3 (E)
- net VCC1.2: now also C11.1, C12.2, C14.1, C3.2 (PLUS), UCT1.4 (OUT); no longer C11.2, C12.1, C14.2, C3.PLUS
- net VCC3.3: now also C10.1, C2.2 (PLUS), R47.1, R48.1, R66.2, UCT2.4 (OUT), TP1.1, U8.4 (VCC); no longer C10.2, C2.PLUS, R47.2, R48.2, R66.1
- net VCC3.3A: now also C22.2 (PLUS), UCT3.4 (OUT); no longer C22.PLUS
- net VCC5: now also C1.2 (PLUS), R65.1, J1.2 (Pin_2); no longer C1.PLUS, R65.2
- net ~{SLT_BUSDIR}: now also R18.1; no longer R11.1
- net ~{SLT_CS12}: now also R24.1; no longer R4.1
- net ~{SLT_CS1}: now also R23.1; no longer R2.1
- net ~{SLT_CS2}: now also R22.1; no longer R3.1
- net ~{SLT_INT}: now also R19.1; no longer R9.1
- net ~{SLT_IORQ}: now also R28.1; no longer R12.1
- net ~{SLT_M1}: now also R27.1; no longer R10.1
- net ~{SLT_MREQ}: now also R17.1; no longer R13.1
- net ~{SLT_RD}: now also R16.1; no longer R15.1
- net ~{SLT_RESET}: now also R30.1; no longer R16.1
- net ~{SLT_RFSH}: now also R20.1; no longer R7.1
- net ~{SLT_SLTSEL}: now also R21.1; no longer R5.1
- net ~{SLT_WAIT}: now also R26.1; no longer R8.1
- net ~{SLT_WR}: now also R29.1; no longer R14.1
- net at R45.1: now also LED1.2 (A); no longer LED1.A
- net at R29.2: now also X1.13; no longer X1.28
- net at R33.2: now also X1.21; no longer X1.32
- net at R6.2: now also X1.34; no longer X1.5
- net at AU1.1 (OUT), AU1.2 (IN-): now also R102.1; no longer R102.2
- net at AU1.3 (IN+), C101.2: now also R101.2; no longer R101.1
- net AV12-: now reaches AU1.4 (VCC-)
- net AV12-: now also AU1.4 (VCC-), AU2.4 (VCC-), AU2.4 (VCC-), C21.1 (MINUS), R55.1
- net AV12+: now reaches AU1.8 (VCC+)
- net AV12+: now also AU1.8 (VCC+), AU2.8 (VCC+), AU2.8 (VCC+), C20.2 (PLUS), R56.1
- net at R2.2: now also X1.42; no longer X1.1
- net at R63.1: now also R61.1, R62.1, T6.K (C); no longer T4.2 (B)
- net at R19.2: now also X1.8; no longer X1.18
- net at C18.2, U2.14 (Vpp/~{WP}): now also R54.2; no longer R54.1
- net at R43.2, U1.53 (VCCA_PLL1): now also C13.2; no longer C13.1
- net at R31.2: now also X1.17; no longer X1.30
- net at D1.2 (K), D2.2 (K), U3.37 (VCC): now also C17.1; no longer C17.2
- net at R32.2: now also X1.19; no longer X1.31
- net at R21.2: now also X1.4; no longer X1.20
- net at U5.15 (AOUTR): now also R201.1; no longer R201.2
- net at U5.16 (AOUTL): now also R101.1; no longer R101.2
- net at C27.2, U5.17 (VCOM): now also C26.2 (PLUS); no longer C26.PLUS
- net at C25.2, R64.2, U5.2 (DVDD)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: now also C23.2 (PLUS); no longer C23.PLUS
- net at R28.2: now also X1.11; no longer X1.27
- net at R37.2: now also X1.29; no longer X1.36
- net at R44.1, U1.157 (VCCA_PLL2): now also C15.1; no longer C15.2
- net at R8.2: now also X1.30; no longer X1.7
- net at R42.2: now also X1.39; no longer X1.42
- net at AU2.6 (IN-), C204.1: now also C203.2 (MINUS), R204.1; no longer C203.MINUS, R204.2
- net at AU2.7 (OUT), C204.2: now also C205.1 (PLUS), R204.2; no longer C205.PLUS, R204.1
- net at XC1.45: now also LED1.1 (K); no longer LED1.K
- net at R13.2: now also X1.20; no longer X1.12
- net at R4.2: now also X1.38; no longer X1.3
- net at D4.2 (K), U3.12 (CE2): now also R50.2; no longer R50.1
- net at AX1.2, AX1.3: now also R205.2, T5.A2 (E); no longer R205.1, T3.3 (E)
- net at AX1.4, AX1.5: now also R105.2, T3.A2 (E); no longer R105.1, T5.3 (E)
- net at R11.2: now also X1.24; no longer X1.10
- net at R12.2: now also X1.22; no longer X1.11
- net at R14.2: now also X1.18; no longer X1.13
- net at X1.14: now also R16.2; no longer R15.2
- net at X1.15: now also R30.2; no longer R16.2
- net at R17.2: now also X1.12; no longer X1.16
- net at R18.2: now also X1.10; no longer X1.17
- net at R20.2: now also X1.6; no longer X1.19
- net at X1.2: now also R22.2; no longer R3.2
- net at R23.2: now also X1.1; no longer X1.22
- net at X1.23: now also R34.2; no longer R24.2
- net at R25.2: now also X1.5; no longer X1.24
- net at X1.25: now also R35.2; no longer R26.2
- net at X1.26: now also R10.2; no longer R27.2
- net at X1.33: now also R39.2; no longer R34.2
- net at R36.2: now also X1.27; no longer X1.35
- net at R38.2: now also X1.31; no longer X1.37
- net at R40.2: now also X1.35; no longer X1.39
- net at R5.2: now also X1.36; no longer X1.4
- net at R41.2: now also X1.37; no longer X1.40
- net at R7.2: now also X1.32; no longer X1.6
- net at R9.2: now also X1.28; no longer X1.8
- net at X1.9: now also R27.2; no longer R10.2
- net at R53.1: now also T1.K (C); no longer T1.1 (C)
- net at R53.2: now also T2.A1 (B); no longer T2.2 (B)
- net at AU2.2 (IN-), C104.1: now also C103.2 (MINUS), R104.1; no longer C103.MINUS, R104.2
- net at R103.1: now also C102.1, R102.2; no longer C103.PLUS
- net at R203.1: now also C202.1, R202.2; no longer C203.PLUS
- net at D2.1 (A): now also R51.2, TP2.1; no longer R51.1
- net at AU2.1 (OUT), C104.2: now also C105.1 (PLUS), R104.2; no longer C105.PLUS, R104.1
- net at U1.121 (nSTATUS): now also R66.1; no longer R66.2
- net at B1.POS: now also R51.1; no longer R51.2
- net at AU1.6 (IN-), AU1.7 (OUT): now also R202.1; no longer R202.2
- removed net +AV12: C20.PLUS, R56.1
- removed net -AV12: C21.MINUS, R55.1
- new net: R63.2, T4.A1 (B)
- new net: C28.2 (PLUS), R60.1, R65.2, T6.A1 (B)
- new net: C29.2 (PLUS), D6.2 (K), T6.A2 (E)
- new net: C205.2 (MINUS), R205.1, R206.1
- new net: R15.2, X1.16
- new net: R24.2, X1.3
- new net: R3.2, X1.40
- new net: R26.2, X1.7
- new net: R52.1, T1.A1 (B)
- new net: R61.2, T3.A1 (B)
- new net: R54.1, T2.K (C)
- new net: C103.1 (PLUS), R103.2
- new net: C203.1 (PLUS), R203.2
- new net: R62.2, T5.A1 (B)
- new net: C105.2 (MINUS), R105.1, R106.1
- new net: AU1.5 (IN+), C201.2, R201.2
Other:
- note removed: "X2"
- note removed: "X3"
- moved on the sheet: B1, D3, D4, R10, R11, R12, R13, R14, R15, R16, R17, R18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

Commit message: Fixed lots of design rule check errors and warnings in pcb Including some serious errors: Lots of fpga GND pins unconnected, C28 connected to wrong net
Connections:
- net HD0 is gone; now on net HD00: XC1.21
- net HD1 is gone; now on net HD01: XC1.22
- net HD2 is gone; now on net HD02: XC1.23
- net HD8 is gone; now on net HD08: XC1.47
- net HD9 is gone; now on net HD09: XC1.48
- net VCC is gone; now on net VCC3.3: C4.2 (PLUS), C5.2, XC1.13, XC1.38
- net ~{HA0} is gone; now on net HA0: U1.179 (IO,_LVDS22n,_DM0T/(DM1T0/BWS#1T0))
- net ~{HA1} is gone; now on net HA1: U1.181 (IO,_LVDS21n)
- net ~{HA2} is gone; now on net HA2: U1.182 (IO,_LVDS21p)
- net ~{HVR} is gone; now on net ~{HWR}: U1.188 (IO,_LVDS20p,_DQ1T1/DQ1T10)
- net GND: now also AX1.M (Mount), XC1.14, XC1.51 (MH1), XC1.52 (MH2), XC1.53 (MH3), XC1.54 (MH4)
- net ~{SLT_RESET}: no longer D5.2 (K)
- net ~{SLT_RESET_RAW}: now reaches R30.2, X1.15
- net ~{SLT_RESET_RAW}: now also D5.2 (K)
Changed lines of the file:
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@@
   (junction (at 452.12 186.69) (diameter 0) (color 0 0 0 0)
   )
+  (junction (at 487.68 224.79) (diameter 0) (color 0 0 0 0)
+  )
   (junction (at 452.12 189.23) (diameter 0) (color 0 0 0 0)
   )
@@
   (junction (at 467.36 118.11) (diameter 0) (color 0 0 0 0)
   )
+  (junction (at 487.68 227.33) (diameter 0) (color 0 0 0 0)
+  )
   (junction (at 396.24 219.71) (diameter 0) (color 0 0 0 0)
   )
+  (junction (at 510.54 189.23) (diameter 0) (color 0 0 0 0)
+  )
   (junction (at 406.4 214.63) (diameter 0) (color 0 0 0 0)
   )
@@
   (junction (at 104.14 212.09) (diameter 0) (color 0 0 0 0)
   )
+  (junction (at 492.76 80.01) (diameter 0) (color 0 0 0 0)
+  )
   (junction (at 452.12 217.17) (diameter 0) (color 0 0 0 0)
   )
@@
   (junction (at 406.4 229.87) (diameter 0) (color 0 0 0 0)
   )
+  (junction (at 487.68 222.25) (diameter 0) (color 0 0 0 0)
+  )
   (junction (at 109.22 349.25) (diameter 0) (color 0 0 0 0)
   )
@@
   (junction (at 152.4 133.35) (diameter 0) (color 0 0 0 0)
   )
+  (junction (at 93.98 273.05) (diameter 0) (color 0 0 0 0)
+  )
   (junction (at 355.6 217.17) (diameter 0) (color 0 0 0 0)
   )
@@
     (stroke (width 0.254) (type default))
   )
+  (wire (pts (xy 487.68 224.79) (xy 487.68 227.33))
+    (stroke (width 0) (type default))
+  )
   (wire (pts (xy 279.4 336.55) (xy 281.94 336.55))
     (stroke (width 0.254) (type default))
@@
     (stroke (width 0.254) (type default))
   )
+  (wire (pts (xy 492.76 80.01) (xy 495.3 80.01))
+    (stroke (width 0) (type default))
+  )
   (wire (pts (xy 111.76 189.23) (xy 114.3 189.23))
     (stroke (width 0.254) (type default))
   )
+  (wire (pts (xy 121.92 274.32) (xy 93.98 274.32))
+    (stroke (width 0) (type default))
+  )
   (wire (pts (xy 472.44 273.05) (xy 452.12 273.05))
     (stroke (width 0.254) (type default))
@@
     (stroke (width 0.254) (type default))
   )
+  (wire (pts (xy 510.54 186.69) (xy 510.54 189.23))
+    (stroke (width 0) (type default))
+  )
   (wire (pts (xy 452.12 166.37) (xy 452.12 168.91))
     (stroke (width 0.254) (type default))
@@
     (stroke (width 0.254) (type default))
   )
+  (wire (pts (xy 93.98 274.32) (xy 93.98 273.05))
+    (stroke (width 0) (type default))
+  )
   (wire (pts (xy 162.56 151.13) (xy 170.18 151.13))
     (stroke (width 0.254) (type default))
@@
     (stroke (width 0.254) (type default))
   )
+  (wire (pts (xy 492.76 80.01) (xy 492.76 77.47))
+    (stroke (width 0.254) (type default))
+  )
   (wire (pts (xy 147.32 143.51) (xy 152.4 143.51))
     (stroke (width 0.254) (type default))
@@
     (stroke (width 0.254) (type default))
   )
+  (wire (pts (xy 487.68 227.33) (xy 487.68 229.87))
+    (stroke (width 0) (type default))
+  )
   (wire (pts (xy 419.1 120.65) (xy 429.26 120.65))
     (stroke (width 0.254) (type default))
@@
     (stroke (width 0.254) (type default))
   )
+  (wire (pts (xy 487.68 219.71) (xy 487.68 222.25))
+    (stroke (width 0) (type default))
+  )
   (wire (pts (xy 492.76 77.47) (xy 495.3 77.47))
     (stroke (width 0.254) (type default))
@@
     (stroke (width 0.254) (type default))
   )
+  (wire (pts (xy 487.68 222.25) (xy 487.68 224.79))
+    (stroke (width 0) (type default))
+  )
   (wire (pts (xy 307.34 219.71) (xy 309.88 219.71))
     (stroke (width 0.254) (type default))
@@
     (stroke (width 0.254) (type default))
   )
-  (wire (pts (xy 492.76 82.55) (xy 492.76 77.47))
+  (wire (pts (xy 492.76 82.55) (xy 492.76 80.01))
     (stroke (width 0.254) (type default))
   )
@@
     (stroke (width 0.254) (type default))
   )
+  (wire (pts (xy 490.22 222.25) (xy 487.68 222.25))
+    (stroke (width 0) (type default))
+  )
   (wire (pts (xy 429.26 92.71) (xy 431.8 92.71))
     (stroke (width 0.254) (type default))
@@
     (stroke (width 0.254) (type default))
   )
+  (wire (pts (xy 490.22 224.79) (xy 487.68 224.79))
+    (stroke (width 0) (type default))
+  )
   (wire (pts (xy 444.5 293.37) (xy 452.12 293.37))
     (stroke (width 0.254) (type default))
@@
     (stroke (width 0.254) (type default))
   )
+  (wire (pts (xy 490.22 219.71) (xy 487.68 219.71))
+    (stroke (width 0) (type default))
+  )
   (wire (pts (xy 256.54 316.23) (xy 254 316.23))
     (stroke (width 0.254) (type default))
@@
     (stroke (width 0.254) (type default))
   )
+  (wire (pts (xy 490.22 227.33) (xy 487.68 227.33))
+    (stroke (width 0) (type default))
+  )
   (wire (pts (xy 256.54 339.09) (xy 254 339.09))
     (stroke (width 0.254) (type default))
@@
     (effects (font (size 1.27 1.27)) (justify right))
   )
+  (hierarchical_label "~{SLT_RESET_RAW}" (shape passive) (at 121.92 274.32 0) (fields_autoplaced)
+    (effects (font (size 1.27 1.27)) (justify left))
+  )
   (hierarchical_label "VCC5" (shape passive) (at 462.28 133.35 270) (fields_autoplaced)
     (effects (font (size 1.27 1.27)) (justify right))
@@
     (effects (font (size 1.27 1.27)) (justify left))
   )
-  (hierarchical_label "HD2" (shape passive) (at 513.08 209.55 0) (fields_autoplaced)
+  (hierarchical_label "HD02" (shape passive) (at 513.08 209.55 0) (fields_autoplaced)
     (effects (font (size 1.27 1.27)) (justify left))
   )
@@
     (effects (font (size 1.27 1.27)) (justify left))
   )
-  (hierarchical_label "VCC" (shape passive) (at 469.9 184.15 180) (fields_autoplaced)
+  (hierarchical_label "VCC3.3" (shape passive) (at 469.9 184.15 180) (fields_autoplaced)
     (effects (font (size 1.27 1.27)) (justify right))
   )
@@
     (effects (font (size 1.27 1.27)) (justify left))
   )
-  (hierarchical_label "~{HVR}" (shape passive) (at 256.54 303.53 0) (fields_autoplaced)
+  (hierarchical_label "~{HWR}" (shape passive) (at 256.54 303.53 0) (fields_autoplaced)
     (effects (font (size 1.27 1.27)) (justify left))
   )
@@
     (effects (font (size 1.27 1.27)) (justify right))
   )
-  (hierarchical_label "HD0" (shape passive) (at 513.08 204.47 0) (fields_autoplaced)
+  (hierarchical_label "HD00" (shape passive) (at 513.08 204.47 0) (fields_autoplaced)
     (effects (font (size 1.27 1.27)) (justify left))
   )
@@
     (effects (font (size 1.27 1.27)) (justify right))
   )
-  (hierarchical_label "HD8" (shape passive) (at 487.68 207.01 180) (fields_autoplaced)
+  (hierarchical_label "HD08" (shape passive) (at 487.68 207.01 180) (fields_autoplaced)
     (effects (font (size 1.27 1.27)) (justify right))
   )
@@
     (effects (font (size 1.27 1.27)) (justify right))
   )
-  (hierarchical_label "~{HA2}" (shape passive) (at 256.54 311.15 0) (fields_autoplaced)
+  (hierarchical_label "HA2" (shape passive) (at 256.54 311.15 0) (fields_autoplaced)
     (effects (font (size 1.27 1.27)) (justify left))
   )
@@
     (effects (font (size 1.27 1.27)) (justify left))
   )
+  (hierarchical_label "GND" (shape passive) (at 487.68 229.87 270) (fields_autoplaced)
+    (effects (font (size 1.27 1.27)) (justify right))
+  )
   (hierarchical_label "SLT_A01" (shape passive) (at 398.78 321.31 0) (fields_autoplaced)
     (effects (font (size 1.27 1.27)) (justify left))
@@
     (effects (font (size 1.27 1.27)) (justify left))
   )
-  (hierarchical_label "VCC" (shape passive) (at 513.08 184.15 0) (fields_autoplaced)
+  (hierarchical_label "VCC3.3" (shape passive) (at 513.08 184.15 0) (fields_autoplaced)
     (effects (font (size 1.27 1.27)) (justify left))
   )
@@
     (effects (font (size 1.27 1.27)) (justify right))
   )
-  (hierarchical_label "~{SLT_RESET}" (shape passive) (at 429.26 128.27 180) (fields_autoplaced)
+  (hierarchical_label "~{SLT_RESET_RAW}" (shape passive) (at 429.26 128.27 180) (fields_autoplaced)
     (effects (font (size 1.27 1.27)) (justify right))
   )
@@
     (effects (font (size 1.27 1.27)) (justify right))
   )
-  (hierarchical_label "HD1" (shape passive) (at 513.08 207.01 0) (fields_autoplaced)
+  (hierarchical_label "HD01" (shape passive) (at 513.08 207.01 0) (fields_autoplaced)
     (effects (font (size 1.27 1.27)) (justify left))
   )
@@
     (effects (font (size 1.27 1.27)) (justify left))
   )
-  (hierarchical_label "HD9" (shape passive) (at 487.68 209.55 180) (fields_autoplaced)
+  (hierarchical_label "HD09" (shape passive) (at 487.68 209.55 180) (fields_autoplaced)
     (effects (font (size 1.27 1.27)) (justify right))
   )
@@
     (effects (font (size 1.27 1.27)) (justify left))
   )
-  (hierarchical_label "~{HA1}" (shape passive) (at 256.54 313.69 0) (fields_autoplaced)
+  (hierarchical_label "HA1" (shape passive) (at 256.54 313.69 0) (fields_autoplaced)
     (effects (font (size 1.27 1.27)) (justify left))
   )
-  (hierarchical_label "~{HA0}" (shape passive) (at 256.54 318.77 0) (fields_autoplaced)
+  (hierarchical_label "HA0" (shape passive) (at 256.54 318.77 0) (fields_autoplaced)
     (effects (font (size 1.27 1.27)) (justify left))
   )
@@
     (pin "2")
     (pin "3")
+    (pin "M")
     (instances
       (project "Carnivore2"

Commit message: Created local footprint library
Connections:
- net AV12+: now also R56.2; no longer R56.1
- net AV12-: now also R55.2; no longer R55.1
- net CONF_DONE: now also R47.1; no longer R47.2
- net GND: now also R50.2; no longer R50.1
- net RSW1: now also R15.2; no longer R15.1
- net RVPPE: now also R52.1; no longer R52.2
- net SLT_A00: now also R9.2; no longer R9.1
- net SLT_A02: now also R8.2; no longer R8.1
- net SLT_A04: now also R7.2; no longer R7.1
- net SLT_A06: now also R12.2; no longer R12.1
- net SLT_A08: now also R11.2; no longer R11.1
- net SLT_A10: now also R13.2; no longer R13.1
- net SLT_A13: now also R10.2; no longer R10.1
- net SLT_A15: now also R14.2; no longer R14.1
- net SLT_CLC: now also R2.2; no longer R2.1
- net SLT_D0: now also R6.2; no longer R6.1
- net SLT_D2: now also R5.2; no longer R5.1
- net SLT_D4: now also R4.2; no longer R4.1
- net SLT_D6: now also R3.2; no longer R3.1
- net VCC+12: now also R56.1; no longer R56.2
- net VCC-12: now also R55.1; no longer R55.2
- net VCC1.2: now also R43.2, R44.1; no longer R43.1, R44.2
- net VCC3.3: now also R45.1, R47.2, R66.1; no longer R45.2, R47.1, R66.2
- net VCC3.3A: now also R64.2; no longer R64.1
- net ~{SLT_BUSDIR}: now also R18.2; no longer R18.1
- net ~{SLT_CS2}: now also R22.2; no longer R22.1
- net ~{SLT_INT}: now also R19.2; no longer R19.1
- net ~{SLT_MREQ}: now also R17.2; no longer R17.1
- net ~{SLT_RD}: now also R16.2; no longer R16.1
- net ~{SLT_RFSH}: now also R20.2; no longer R20.1
- net ~{SLT_SLTSEL}: now also R21.2; no longer R21.1
- net at LED1.2 (A): now also R45.2; no longer R45.1
- net at X1.34: now also R6.1; no longer R6.2
- net at X1.42: now also R2.1; no longer R2.2
- net at R61.1, T6.K (C): now also R62.2, R63.2; no longer R62.1, R63.1
- net at T4.A1 (B): now also R63.1; no longer R63.2
- net at X1.8: now also R19.1; no longer R19.2
- net at C18.2, U2.14 (Vpp/~{WP}): now also R54.1; no longer R54.2
- net at C13.2, U1.53 (VCCA_PLL1): now also R43.1; no longer R43.2
- net at X1.4: now also R21.1; no longer R21.2
- net at C23.2 (PLUS), C25.2, U5.2 (DVDD)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: now also R64.1; no longer R64.2
- net at C15.1, U1.157 (VCCA_PLL2): now also R44.2; no longer R44.1
- net at X1.30: now also R8.1; no longer R8.2
- net at X1.20: now also R13.1; no longer R13.2
- net at X1.38: now also R4.1; no longer R4.2
- net at D4.2 (K), U3.12 (CE2): now also R50.1; no longer R50.2
- net at X1.24: now also R11.1; no longer R11.2
- net at X1.10: now also R18.1; no longer R18.2
- net at X1.12: now also R17.1; no longer R17.2
- net at X1.14: now also R16.1; no longer R16.2
- net at X1.16: now also R15.1; no longer R15.2
- net at X1.18: now also R14.1; no longer R14.2
- net at X1.2: now also R22.1; no longer R22.2
- net at X1.22: now also R12.1; no longer R12.2
- net at X1.26: now also R10.1; no longer R10.2
- net at X1.28: now also R9.1; no longer R9.2
- net at X1.32: now also R7.1; no longer R7.2
- net at X1.36: now also R5.1; no longer R5.2
- net at X1.40: now also R3.1; no longer R3.2
- net at X1.6: now also R20.1; no longer R20.2
- net at T1.A1 (B): now also R52.2; no longer R52.1
- net at T1.K (C): now also R53.2; no longer R53.1
- net at T2.A1 (B): now also R53.1; no longer R53.2
- net at T2.K (C): now also R54.2; no longer R54.1
- net at T5.A1 (B): now also R62.1; no longer R62.2
- net at D2.1 (A), TP2.1: now also R51.1; no longer R51.2
- net at U1.121 (nSTATUS): now also R66.2; no longer R66.1
- net at B1.POS: now also R51.2; no longer R51.1
Other:
- moved on the sheet: R10, R11, R12, R13, R14, R15, R16, R17, R18, R19, R2, R20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
