File: Board/Carnivore2.kicad_sch (KiCad schematic)
At the start: 135 parts, among them J1 Conn_01x02_Pin, J2 Conn_01x03_Pin, U1 EP2C8Q208C8N, U2 MX29LV640ETTI-70G, U3 RMLV1616AGSA-5S#KA0, U4 M25P80-VMN3TPB, U5 PCM5101APWR, U6 AT93C46DN-SH-T, U7 SG3225CAN 50.0000M-TJGA6, U9 PCM1808PWR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

Commit message: Hardware modification to delay Z80 startup until FPGA is configured Needed on FS-A1W(S)X models
Parts:
- added Q1: MMBT3904-TP, Package_TO_SOT_SMD:SOT-23, symbol Transistor_BJT:MMBT2222A
- added R52: 10k, Resistor_SMD:R_0603_1608Metric, symbol Sheet1-altium-import:root_2_R_0805
- added R53, R54: 4k7, Resistor_SMD:R_0603_1608Metric, symbol Sheet1-altium-import:root_2_R_0805
- J2: value Conn_01x03_Pin -> Conn_01x05_Pin; footprint Connector_PinHeader_2.54mm:PinHeader_1x03_P2.54mm_Vertical -> Connector_PinHeader_2.54mm:PinHeader_1x05_P2.54mm_Vertical; symbol Connector:Conn_01x03_Pin -> Connector:Conn_01x05_Pin
Connections:
- net GND: now also Q1.2 (E), R52.2
- net VCC3.3: now also R53.1
- net ~{SLT_WAIT}: now also Q1.3 (C)
- net at J2.2 (Pin_2): now also U1.45 (IO,_LVDS0n); no longer U1.44 (IO,_LVDS0p)
- net at J2.3 (Pin_3): now also U1.46 (IO); no longer U1.45 (IO,_LVDS0n)
- net at U1.47 (IO,_PLL1_OUTp): now also J2.4 (Pin_4)
- net at U1.48 (IO,_PLL1_OUTn): now also J2.5 (Pin_5)
- new net: Q1.1 (B), R52.1, R54.2
- new net ~{SLT_READY}: R53.2, R54.1, U1.44 (IO,_LVDS0p)
Other:
- note added: "Hold the bus until ~{SLT_READY} gets asserted by the FPGA This allows the FPGA to boot before the MSX BIOS scans the slots"

Commit message: Minor improvements
Connections:
- net VCC1.2 renamed +1V2
- net VCC3.3 renamed +3.3V
- net VCC3.3A renamed +3.3VDAC
- net VCC5 renamed +5V
Changed lines of the file:
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@@
 		)
 	)
-	(hierarchical_label "VCC3.3"
+	(hierarchical_label "+3.3V"
 		(shape passive)
 		(at 500.38 300.99 180)
@@
 		)
 	)
-	(hierarchical_label "VCC3.3"
+	(hierarchical_label "+3.3V"
 		(shape passive)
 		(at 469.9 341.63 180)
@@
 		)
 	)
-	(hierarchical_label "VCC3.3"
+	(hierarchical_label "+3.3V"
 		(shape passive)
 		(at 469.9 184.15 180)
@@
 		)
 	)
-	(hierarchical_label "VCC3.3"
+	(hierarchical_label "+3.3V"
 		(shape passive)
 		(at 515.62 237.49 0)
@@
 		)
 	)
-	(hierarchical_label "VCC3.3"
+	(hierarchical_label "+3.3V"
 		(shape passive)
 		(at 185.42 234.95 0)
@@
 		)
 	)
-	(hierarchical_label "VCC3.3"
+	(hierarchical_label "+3.3V"
 		(shape passive)
 		(at 500.38 307.34 180)
@@
 		)
 	)
-	(hierarchical_label "VCC3.3"
+	(hierarchical_label "+3.3V"
 		(shape passive)
 		(at 317.5 196.85 0)
@@
 		)
 	)
-	(hierarchical_label "VCC3.3"
+	(hierarchical_label "+3.3V"
 		(shape passive)
 		(at 393.7 237.49 180)
@@
 		)
 	)
-	(hierarchical_label "VCC5"
+	(hierarchical_label "+5V"
 		(shape passive)
 		(at 259.08 219.71 180)
@@
 		)
 	)
-	(hierarchical_label "VCC3.3"
+	(hierarchical_label "+3.3V"
 		(shape passive)
 		(at 486.41 322.58 180)
@@
 		)
 	)
-	(hierarchical_label "VCC1.2"
+	(hierarchical_label "+1V2"
 		(shape passive)
 		(at 317.5 222.25 0)
@@
 		)
 	)
-	(hierarchical_label "VCC3.3"
+	(hierarchical_label "+3.3V"
 		(shape passive)
 		(at 154.94 133.35 0)
@@
 		)
 	)
-	(hierarchical_label "VCC5"
+	(hierarchical_label "+5V"
 		(shape passive)
 		(at 265.43 242.57 180)
@@
 		)
 	)
-	(hierarchical_label "VCC3.3"
+	(hierarchical_label "+3.3V"
 		(shape passive)
 		(at 142.24 54.61 0)
@@
 		)
 	)
-	(hierarchical_label "VCC3.3"
+	(hierarchical_label "+3.3V"
 		(shape passive)
 		(at 170.18 191.77 270)
@@
 		)
 	)
-	(hierarchical_label "VCC3.3"
+	(hierarchical_label "+3.3V"
 		(shape passive)
 		(at 80.01 180.34 180)
@@
 		)
 	)
-	(hierarchical_label "VCC3.3"
+	(hierarchical_label "+3.3V"
 		(shape passive)
 		(at 513.08 184.15 0)
@@
 		)
 	)
-	(hierarchical_label "VCC3.3"
+	(hierarchical_label "+3.3V"
 		(shape passive)
 		(at 264.795 41.91 180)
@@
 		)
 	)
-	(hierarchical_label "VCC3.3"
+	(hierarchical_label "+3.3V"
 		(shape passive)
 		(at 241.3 133.35 0)
@@
 		)
 	)
-	(hierarchical_label "VCC3.3"
+	(hierarchical_label "+3.3V"
 		(shape passive)
 		(at 452.12 295.91 270)
@@
 		)
 	)
-	(hierarchical_label "VCC3.3A"
+	(hierarchical_label "+3.3VDAC"
 		(shape passive)
 		(at 317.5 171.45 0)
@@
 		)
 	)
-	(hierarchical_label "VCC3.3"
+	(hierarchical_label "+3.3V"
 		(shape passive)
 		(at 447.04 334.01 0)
@@
 		)
 	)
-	(hierarchical_label "VCC1.2"
+	(hierarchical_label "+1V2"
 		(shape passive)
 		(at 370.84 161.29 180)
@@
 		)
 	)
-	(hierarchical_label "VCC5"
+	(hierarchical_label "+5V"
 		(shape passive)
 		(at 280.035 36.195 180)
@@
 		)
 	)
-	(hierarchical_label "VCC3.3A"
+	(hierarchical_label "+3.3VDAC"
 		(shape passive)
 		(at 481.33 36.83 0)
@@
 		)
 	)
-	(hierarchical_label "VCC3.3"
+	(hierarchical_label "+3.3V"
 		(shape passive)
 		(at 510.54 290.83 270)
@@
 		)
 	)
-	(hierarchical_label "VCC5"
+	(hierarchical_label "+5V"
 		(shape passive)
 		(at 96.52 350.52 0)
@@
 		)
 	)
-	(hierarchical_label "VCC1.2"
+	(hierarchical_label "+1V2"
 		(shape passive)
 		(at 401.32 148.59 90)
@@
 		)
 	)
-	(hierarchical_label "VCC3.3A"
+	(hierarchical_label "+3.3VDAC"
 		(shape passive)
 		(at 483.87 87.63 0)
@@
 		)
 	)
-	(hierarchical_label "VCC1.2"
+	(hierarchical_label "+1V2"
 		(shape passive)
 		(at 354.33 181.61 180)

Commit message: Improved slot wait
Parts:
- R53: DIGIKEY RMCF0603FT10K0CT-ND -> RMCF0603FT4K70CT-ND
- R54: value 4k7 -> 470E; DIGIKEY RMCF0603FT10K0CT-ND -> RMCF0603FT470RCT-ND
Connections:
- net ~{SLT_WAIT}: no longer Q1.3 (C)
- net ~{X_SLT_WAIT}: now reaches R26.2, X1.7
- net ~{X_SLT_WAIT}: now also Q1.3 (C)
Other:
- moved on the sheet: R26
Changed lines of the file:
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@@
 	(wire
 		(pts
-			(xy 78.74 254) (xy 81.28 254)
-		)
-		(stroke
-			(width 0.254)
-			(type default)
-		)
-	)
-	(wire
-		(pts
 			(xy 215.9 146.05) (xy 215.9 143.51)
 		)
@@
 	(wire
 		(pts
-			(xy 93.98 254) (xy 91.44 254)
+			(xy 93.98 232.41) (xy 91.44 232.41)
 		)
 		(stroke
@@
 	(wire
 		(pts
+			(xy 78.74 254) (xy 93.98 254)
+		)
+		(stroke
+			(width 0)
+			(type default)
+		)
+	)
+	(wire
+		(pts
 			(xy 147.32 87.63) (xy 144.78 87.63)
 		)
@@
 	(hierarchical_label "~{SLT_WAIT}"
 		(shape passive)
-		(at 93.98 254 0)
+		(at 93.98 232.41 0)
 		(effects
 			(font
@@
 		)
 	)
-	(hierarchical_label "~{SLT_WAIT}"
+	(hierarchical_label "~{X_SLT_WAIT}"
 		(shape passive)
 		(at 92.71 200.66 0)
@@
 		)
 	)
+	(hierarchical_label "~{X_SLT_WAIT}"
+		(shape passive)
+		(at 93.98 254 0)
+		(effects
+			(font
+				(size 1.27 1.27)
+			)
+			(justify left)
+		)
+	)
 	(hierarchical_label "GND"
 		(shape passive)
@@
 		)
 	)
+	(hierarchical_label "~{X_SLT_WAIT}"
+		(shape passive)
+		(at 81.28 232.41 180)
+		(effects
+			(font
+				(size 1.27 1.27)
+			)
+			(justify right)
+		)
+	)
 	(hierarchical_label "~{SLT_M1}"
 		(shape passive)
@@
 			)
 		)
-		(property "DIGIKEY" "RMCF0603FT10K0CT-ND"
+		(property "DIGIKEY" "RMCF0603FT4K70CT-ND"
 			(at 82.55 184.15 0)
 			(effects
@@
 	(symbol
 		(lib_id "Sheet1-altium-import:root_2_R_0805")
-		(at 91.44 254 0)
+		(at 91.44 232.41 0)
 		(unit 1)
 		(exclude_from_sim no)
@@
 		(dnp no)
 		(property "Reference" "R26"
-			(at 81.28 252.73 0)
+			(at 86.106 229.362 0)
 			(effects
 				(font
@@
 		)
 		(property "Value" "330E"
-			(at 91.44 254 0)
+			(at 91.44 232.41 0)
 			(effects
 				(font
@@
 		)
 		(property "Footprint" "Resistor_SMD:R_0603_1608Metric"
-			(at 91.44 254 0)
+			(at 91.44 232.41 0)
 			(effects
 				(font
@@
 		)
 		(property "Datasheet" ""
-			(at 91.44 254 0)
+			(at 91.44 232.41 0)
 			(effects
 				(font
@@
 		)
 		(property "Description" ""
-			(at 91.44 254 0)
+			(at 91.44 232.41 0)
 			(effects
 				(font
@@
 		)
 		(property "DIGIKEY" "RMCF0603FT330RCT-ND"
-			(at 91.44 254 0)
+			(at 91.44 232.41 0)
 			(effects
 				(font
@@
 			)
 		)
-		(property "Value" "4k7"
+		(property "Value" "470E"
 			(at 83.82 200.66 0)
 			(effects
@@
 			)
 		)
-		(property "DIGIKEY" "RMCF0603FT10K0CT-ND"
+		(property "DIGIKEY" "RMCF0603FT470RCT-ND"
 			(at 82.55 196.85 0)
 			(effects
